File: blinkey.kicad_sch (KiCad schematic)
At the start: 34 parts, among them SW1 SW_DIP_x04

Commit message: Adding USB-C
Parts:
- LCD1: footprint st7789:st7789 -> Connector_PinSocket_2.54mm:PinSocket_1x08_P2.54mm_Vertical_SMD_Pin1Left
Changed lines of the file:
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@@
   (title_block
     (title "ULX3S")
-    (rev "1.0.3")
+    (date "2023-01-19")
+    (rev "3.1.8")
     (company "EMARD")
     (comment 1 "Buttons, LEDs, OLED display")
@@
     (property "Reference" "LCD1" (id 0) (at 110.49 39.37 0))
     (property "Value" "ST7789" (id 1) (at 107.95 39.37 0))
-    (property "Footprint" "st7789:st7789" (id 2) (at 115.57 39.37 90)
-      (effects (font (size 1.27 1.27)) hide)
-    )
+    (property "Footprint" "Connector_PinSocket_2.54mm:PinSocket_1x08_P2.54mm_Vertical_SMD_Pin1Left" (id 2) (at 115.57 39.37 90)
+      (effects (font (size 1.27 1.27)) hide)
+    )
